File: Schematics/Team16_FINAL.sch (EAGLE design)
At the start: 20 parts, among them J1 AVR_SPI_PROG_3X2PTH, U1 ATMEGA328P_TQFP, U3 ADXL345, U4 3.3V/150mA, Y1 8MHz

Commit message: Add files via upload
Parts:
- added R1, R2, R3, R4: 0, SparkFun-Resistors:0OHM-0402-1/10W
- C4: device SparkFun-Capacitors:0.1UF-0603-25V-(+80/-20%) -> SparkFun-Capacitors:0.1UF-0402-16V-10%
Connections:
- new net N$5: R1.1, U3.CS
- new net N$6: R2.1, U3.SDO
- new net N$7: R3.1, U3.SDA
- new net N$9: R4.1, U3.SCL
- net MISO: now also R2.2; no longer U3.SDO
- net MOSI: now also R3.2; no longer U3.SDA
- net N$14: now also R1.2; no longer U3.CS
- net SCK: now also R4.2; no longer U3.SCL
